File: Hardware/Driver_motor_board/Driver_motor.kicad_pcb (KiCad board)
At the start: 2 copper layers, 78.5 x 90.2 mm, 74 parts, among them J1 B6B-XH-A(LF)(SN), J2 B6B-XH-A(LF)(SN), J3 B9B-XH-A(LF)(SN), J4 B6B-XH-A(LF)(SN), J5 B6B-XH-A(LF)(SN), J6 B8B-XH-A(LF)(SN), J7 282814-2, J8 282814-2, U1 BTS7960B, U10 BTS7960B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

Commit message: add main board
Other:
- board text added: "."
- board text added: "ENCODER M1A->M4B"
- board text added: "PWM GND-M4->M1"
- board text removed: "ENCODER M1->M4"
- board text removed: "GND M4->M1"
Changed lines of the file:
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@@
     (effects (font (size 1 1) (thickness 0.15)))
   )
-  (gr_text "ENCODER M1->M4" (at 79.502 67.31 90) (layer "F.SilkS")
+  (gr_text "ENCODER M1A->M4B" (at 79.502 67.31 90) (layer "F.SilkS")
     (effects (font (size 1 1) (thickness 0.15)))
   )
@@
     (effects (font (size 0.787402 0.787402) (thickness 0.15)))
   )
+  (gr_text "." (at 132.334 80.772) (layer "F.SilkS")
+    (effects (font (size 5 5) (thickness 0.15)))
+  )
   (gr_text "+" (at 89.916 92.456 180) (layer "F.SilkS")
     (effects (font (size 0.787402 0.787402) (thickness 0.15)))
   )
-  (gr_text "GND M4->M1" (at 140.716 101.346 90) (layer "F.SilkS")
+  (gr_text "PWM GND-M4->M1" (at 140.716 101.346 90) (layer "F.SilkS")
     (effects (font (size 1 1) (thickness 0.15)))
   )
@@
     (effects (font (size 1 1) (thickness 0.15)))
   )
+  (dimension (type aligned) (layer "F.SilkS")
+    (pts (xy 70.231 131.826) (xy 148.844 131.826))
+    (height 5.334)
+    (gr_text "3095.0000 mils" (at 109.5375 136.01) (layer "F.SilkS")
+      (effects (font (size 1 1) (thickness 0.15)))
+    )
+    (format (prefix "") (suffix "") (units 3) (units_format 1) (precision 4))
+    (style (thickness 0.15) (arrow_length 1.27) (text_position_mode 0) (extension_height 0.58642) (extension_offset 0.5) keep_text_aligned)
+  )
+  (dimension (type aligned) (layer "F.SilkS")
+    (pts (xy 148.717 41.656) (xy 148.717 132.08))
+    (height -14.097)
+    (gr_text "3560.0000 mils" (at 161.664 86.868 90) (layer "F.SilkS")
+      (effects (font (size 1 1) (thickness 0.15)))
+    )
+    (format (prefix "") (suffix "") (units 3) (units_format 1) (precision 4))
+    (style (thickness 0.15) (arrow_length 1.27) (text_position_mode 0) (extension_height 0.58642) (extension_offset 0.5) keep_text_aligned)
+  )
   (segment (start 95.25 53.34) (end 95.25 50.4005) (width 0.762) (layer "F.Cu") (net 1))
