Commit message: pussh

File: install/bbb_robot/share/bbb_robot/description/gazebo_control.xacro (robot description, xacro)
@@ -1 +1,31 @@
-/home/jetson/bbb_jetson_ws/src/bbb_robot/description/gazebo_control.xacro
+<?xml version="1.0"?>
+<robot xmlns:xacro="http://www.ros.org/wiki/xacro">
+    <gazebo>
+        <plugin name="diff_drive" filename="libgazebo_ros_diff_drive.so">  <!-- filename is the name
+            plugin used-->
+            <!-- WHEEL BACK INFORMATION-->
+            <left_joint>left_wheel_back_joint </left_joint>
+            <right_joint>right_wheel_back_joint</right_joint>
+            <wheel_separation>0.232</wheel_separation>
+            <wheel_diameter> 0.125</wheel_diameter>
+            <!-- WHEEL FOWARDD INFORMATION-->
+            <!-- <left_joint>left_wheel_foward_joint </left_joint>
+            <right_joint>right_wheel__joint</right_joint>
+            <wheel_separation>0.232</wheel_separation>
+            <wheel_diameter> 0.125</wheel_diameter> -->
+            <!-- LIMITS-->
+            <max_wheel_torque>200</max_wheel_torque>
+            <max_wheel_acceleration> 10.0</max_wheel_acceleration>
+            <!-- OUTPUTS-->
+            <odometry_frame>odom</odometry_frame>
+            <robot_base_frame>base_footprint</robot_base_frame><!-- standard link-->
+            <publish_odom>true</publish_odom><!-- publish odom if had message "true"-->
+            <publish_odom_tf>true</publish_odom_tf>
+            <publish_wheel_tf>true</publish_wheel_tf>
+        </plugin>
+    </gazebo>
+</robot>
+<!-- ros2 run teleop_twist_keyboard teleop_twist_keyboard -->
+<!-- teleop: stands for teleoperation
+twist: type of date, ros uused to express linear velocity and angle
+keyboard: use keyboard to control remote robot -->

File: install/bbb_robot/share/bbb_robot/description/inertial_macros.xacro (robot description, xacro)
@@ -1 +1,33 @@
-/home/jetson/bbb_jetson_ws/src/bbb_robot/description/inertial_macros.xacro
+<?xml version="1.0"?>
+<robot xmlns:xacro="http://www.ros.org/wiki/xacro">
+    <!-- Specify some standard inertial calculations
+    https://en.wikipedia.org/wiki/List_of_moments_of_inertia -->
+    <!-- These make use of xacro's mathematical functionality -->
+    <xacro:macro name="inertial_sphere" params="mass radius *origin">
+        <inertial>
+            <xacro:insert_block name="origin" />
+            <mass value="${mass}" />
+            <inertia ixx="${(2/5) * mass * (radius*radius)}" ixy="0.0" ixz="0.0"
+                iyy="${(2/5) * mass * (radius*radius)}" iyz="0.0"
+                izz="${(2/5) * mass * (radius*radius)}" />
+        </inertial>
+    </xacro:macro>
+    <xacro:macro name="inertial_box" params="mass x y z *origin">
+        <inertial>
+            <xacro:insert_block name="origin" />
+            <mass value="${mass}" />
+            <inertia ixx="${(1/12) * mass * (y*y+z*z)}" ixy="0.0" ixz="0.0"
+                iyy="${(1/12) * mass * (x*x+z*z)}" iyz="0.0"
+                izz="${(1/12) * mass * (x*x+y*y)}" />
+        </inertial>
+    </xacro:macro>
+    <xacro:macro name="inertial_cylinder" params="mass length radius *origin">
+        <inertial>
+            <xacro:insert_block name="origin" />
+            <mass value="${mass}" />
+            <inertia ixx="${(1/12) * mass * (3*radius*radius + length*length)}" ixy="0.0" ixz="0.0"
+                iyy="${(1/12) * mass * (3*radius*radius + length*length)}" iyz="0.0"
+                izz="${(1/2) * mass * (radius*radius)}" />
+        </inertial>
+    </xacro:macro>
+</robot>

File: install/bbb_robot/share/bbb_robot/description/lidar2D.xacro (robot description, xacro)
@@ -1 +1,56 @@
-/home/jetson/bbb_jetson_ws/src/bbb_robot/description/lidar2D.xacro
+<?xml version="1.0"?>
+<robot xmlns:xacro="http://www.ros.org/wiki/xacro">
+    <joint name="lidar2D_joint" type="fixed">
+        <parent link="base_link" />
+        <child link="lidar2D_frame" />
+        <origin xyz="-0.052 0.0 0.12" rpy="0.0 0.0 0.0" />
+    </joint>
+    <link name="lidar2D_frame">
+        <visual>
+            <geometry>
+                <cylinder radius="0.035" length="0.04" />
+            </geometry>
+            <material name="red" />
+        </visual>
+        <collision>
+            <geometry>
+                <cylinder radius="0.035" length="0.04" />
+            </geometry>
+            <!-- <material name="orange" /> -->
+        </collision>
+        <xacro:inertial_cylinder mass="0.1" length="0.04" radius="0.05">
+            <origin xyz="0 0 0" rpy="0 0 0" />
+        </xacro:inertial_cylinder>
+    </link>
+    <gazebo reference="lidar2D_frame">
+        <material>Gazebo/Red</material>
+        <sensor name="lidar2D" type="ray">
+            <pose> 0 0 0 0 0 0 </pose> <!-- origin sensor is in origin of lidar2D_frame-->
+            <visualize>true</visualize> <!-- display sensor in gazebo-->
+            <update_rate>10</update_rate> <!-- update data from sensor 10 times/sencond-->
+            <ray><!-- paramettor of ray sensor-->
+                <scan>
+                    <horizontal><!-- scan horizontally-->
+                        <samples>360</samples>
+                        <resolution>1</resolution>
+                        <min_angle>-3.14</min_angle>
+                        <max_angle>3.14</max_angle>
+                    </horizontal>
+                </scan>
+                <range>
+                    <min>0.3</min>
+                    <max>12</max>
+                    <resolution>0.01</resolution>
+                </range>
+            </ray>
+            <plugin name="lidar2D_controller" filename="libgazebo_ros_ray_sensor.so">
+                <!-- plugin is the thing that gazebo interact with the thing outside gazebo-->
+                <ros>
+                    <argument>~/out:=scan</argument> <!-- topic scan-->
+                </ros>
+                <output_type>sensor_msgs/LaserScan</output_type>
+                <frame_name>lidar2D_frame</frame_name>
+            </plugin>
+        </sensor>
+    </gazebo>
+</robot>

File: install/bbb_robot/share/bbb_robot/description/robot.urdf.xacro (robot description, xacro)
@@ -1 +1,13 @@
-/home/jetson/bbb_jetson_ws/src/bbb_robot/description/robot.urdf.xacro
+<?xml version="1.0"?>
+<robot xmlns:xacro="http://www.ros.org/wiki/xacro" name="robot">
+    <!-- <xacro:include filename="robot_core_differential_robot.xacro" /> -->
+    <xacro:include filename="robot_core_four_wheel.xacro" />
+    <!-- <xacro:arg name="use_ros2_control" default="true" />
+    <xacro:if value="$(arg use_ros2_control)">
+        <xacro:include filename="ros2_control.xacro" />
+    </xacro:if>
+    <xacro:unless value="$(arg use_ros2_control)">
+        <xacro:include filename="gazebo_control.xacro" />
+    </xacro:unless> -->
+    <xacro:include filename="lidar2D.xacro" />
+</robot>

File: install/bbb_robot/share/bbb_robot/description/robot_core_differential_robot.xacro (robot description, xacro)
@@ -1 +1,138 @@
-/home/jetson/bbb_jetson_ws/src/bbb_robot/description/robot_core_differential_robot.xacro
+<?xml version="1.0"?>
+<robot xmlns:xacro="http://www.ros.org/wiki/xacro">
+    <xacro:include filename="inertial_macros.xacro" />
+    <material name="white">
+        <color rgba="1 1 1 1" />
+    </material>
+    <material name="orange">
+        <color rgba="1 0.3 0.1 1" />
+    </material>
+    <material name="blue">
+        <color rgba="0.2 0.2 1 1" />
+    </material>
+    <material name="black">
+        <color rgba="0 0 0 1" />
+    </material>
+    <material name="red">
+        <color rgba="1 0 0 1" />
+    </material>
+    <!--BASE
+    FOOTPRINT-->
+    <link name="base_footprint">
+    </link>
+    <!--BASE
+    LINK-->
+    <joint name="base_joint" type="fixed">
+        <parent link="base_footprint" />
+        <child link="base_link" />
+        <origin xyz="0 0 0.0625" />
+    </joint>
+    <link name="base_link">
+        <visual>
+            <origin xyz="0 0.0 0.06" /><!-- 0.12/2 -->
+            <geometry>
+                <box size="0.25 0.18 0.12" />
+            </geometry>
+            <material name="white" />
+        </visual>
+        <collision>
+            <origin xyz="0 0.0 0.06" /><!-- 0.12/2-->
+            <geometry>
+                <box size="0 0.18 0.12" />
+            </geometry>
+            <!-- <material name="black" /> -->
+        </collision>
+        <xacro:inertial_box mass="0.5" x="0.3" y="0.3" z="0.15">
+            <origin xyz="0 0.0 0.06" rpy="0 0 0" />
+        </xacro:inertial_box>
+    </link>
+    <gazebo reference="base_link">
+        <material>Gazebo/Purple</material>
+    </gazebo>
+    <!--LEFT
+    WHEEL BACK LINK-->
+    <joint name="left_wheel_back_joint" type="continuous">
+        <parent link="base_link" />
+        <child link="left_wheel_back_link" />
+        <origin
+            xyz="-0.075 0.116 0.0" rpy="-${pi/2} 0.0 0.0" /><!-- 116 = 90+52/2-->
+        <axis xyz="0.0 0.0 1" />
+    </joint>
+    <link name="left_wheel_back_link">
+        <visual>
+            <geometry>
+                <cylinder radius="0.0625" length="0.05132" />
+            </geometry>
+            <material name="blue" />
+        </visual>
+        <collision>
+            <geometry>
+                <!-- <cylinder radius="0.0625" length="0.05132" /> -->
+                <sphere radius="0.0625" />
+            </geometry>
+            <!-- <material name="orange" /> -->
+        </collision>
+        <xacro:inertial_cylinder mass="0.1" length="0.04" radius="0.05">
+            <origin xyz="0 0 0" rpy="0 0 0" />
+        </xacro:inertial_cylinder>
+    </link>
+    <gazebo reference="left_wheel_back_link">
+        <material>Gazebo/Blue</material>
+    </gazebo>
+    <!--RIGHT
+    WHEEL BACK LINK-->
+    <joint name="right_wheel_back_joint" type="continuous">
+        <parent link="base_link" />
+        <child link="right_wheel_back_link" />
+        <origin xyz="-0.075 -0.116 0.0" rpy="${pi/2} 0.0 0.0" /><!-- 116 = 90+52/2-->
+        <axis xyz="0.0 0.0 -1" />
+    </joint>
+    <link name="right_wheel_back_link">
+        <visual>
+            <geometry>
+                <cylinder radius="0.0625" length="0.05132" />
+            </geometry>
+            <material name="blue" />
+        </visual>
+        <collision>
+            <geometry>
+                <!-- <cylinder radius="0.0625" length="0.05132" /> -->
+                <sphere radius="0.0625" />
+            </geometry>
+            <!-- <material name="orange" /> -->
+        </collision>
+        <xacro:inertial_cylinder mass="0.1" length="0.04" radius="0.05">
+            <origin xyz="0 0 0" rpy="0 0 0" />
+        </xacro:inertial_cylinder>
+    </link>
+    <gazebo reference="right_wheel_back_link">
+        <material>Gazebo/Blue</material>
+    </gazebo>
+    <!-- CASTER WHEEL LINK -->
+    <joint name="caster_wheel_joint" type="fixed">
+        <parent link="base_link" />
+        <child link="caster_wheel_link" />
+        <origin xyz="0.06 0 0.0" />
+    </joint>
+    <link name="caster_wheel_link">
+        <visual>
+            <geometry>
+                <sphere radius="0.0625" />
+            </geometry>
+            <material name="black" />
+        </visual>
+        <collision>
+            <geometry>
+                <sphere radius="0.0625" />
+            </geometry>
+        </collision>
+        <xacro:inertial_sphere mass="0.1" radius="0.0625">
+            <origin xyz="0 0 0" rpy="0 0 0" />
+        </xacro:inertial_sphere>
+    </link>
+    <gazebo reference="caster_wheel_link">
+        <material>Gazebo/Black</material>
+        <mu1 value="0.002" />
+        <mu2 value="0.002" />
+    </gazebo>
+</robot>

File: install/bbb_robot/share/bbb_robot/description/robot_core_four_wheel.xacro (robot description, xacro)
@@ -1 +1,172 @@
-/home/jetson/bbb_jetson_ws/src/bbb_robot/description/robot_core_four_wheel.xacro
+<?xml version="1.0"?>
+<robot xmlns:xacro="http://www.ros.org/wiki/xacro">
+    <xacro:include filename="inertial_macros.xacro" />
+    <material name="white">
+        <color rgba="1 1 1 1" />
+    </material>
+    <material name="orange">
+        <color rgba="1 0.3 0.1 1" />
+    </material>
+    <material name="blue">
+        <color rgba="0.2 0.2 1 1" />
+    </material>
+    <material name="black">
+        <color rgba="0 0 0 1" />
+    </material>
+    <material name="red">
+        <color rgba="1 0 0 1" />
+    </material>
+    <!--BASE
+    FOOTPRINT-->
+    <link name="base_footprint">
+    </link>
+    <!--BASE
+    LINK-->
+    <joint name="base_joint" type="fixed">
+        <parent link="base_footprint" />
+        <child link="base_link" />
+        <origin xyz="0 0 0.0625" />
+    </joint>
+    <link name="base_link">
+        <visual>
+            <origin xyz="0 0.0 0.06" /><!-- 0.12/2 -->
+            <geometry>
+                <box size="0.25 0.18 0.12" />
+            </geometry>
+            <material name="white" />
+        </visual>
+        <collision>
+            <origin xyz="0 0.0 0.06" /><!-- 0.12/2-->
+            <geometry>
+                <box size="0 0.18 0.12" />
+            </geometry>
+            <!-- <material name="black" /> -->
+        </collision>
+        <xacro:inertial_box mass="0.5" x="0.3" y="0.3" z="0.15">
+            <origin xyz="0 0.0 0.06" rpy="0 0 0" />
+        </xacro:inertial_box>
+    </link>
+    <gazebo reference="base_link">
+        <material>Gazebo/Purple</material>
+    </gazebo>
+    <!--LEFT
+    WHEEL BACK LINK-->
+    <joint name="left_wheel_back_joint" type="fixed">
+        <parent link="base_link" />pe="continuo <child link="left_wheel_back_link" />
+        <origin
+            xyz="-0.075 0.116 0.0" rpy="-${pi/2} 0.0 0.0" /><!-- 116 = 90+52/2-->
+        <axis xyz="0.0 0.0 1" />
+    </joint>
+    <link name="left_wheel_back_link">
+        <visual>
+            <geometry>
+                <cylinder radius="0.0625" length="0.05132" />
+            </geometry>
+            <material name="blue" />
+        </visual>
+        <collision>
+            <geometry>
+               <sphere radius="0.0625" />
+                <!-- <cylinder radius="0.0625" length="0.05132" /> -->
+            </geometry>
+            <!-- <material name="orange" /> -->
+        </collision>
+        <xacro:inertial_cylinder mass="0.1" length="0.04" radius="0.05">
+            <origin xyz="0 0 0" rpy="0 0 0" />
+        </xacro:inertial_cylinder>
+    </link>
+    <gazebo reference="left_wheel_back_link">
+        <material>Gazebo/Blue</material>
+    </gazebo>
+    <!--RIGHT
+    WHEEL BACK LINK-->
+    <joint name="right_wheel_back_joint" type="fixed">
+        <parent link="base_link" />
+        <child link="right_wheel_back_link" />
+        <origin xyz="-0.075 -0.116 0.0" rpy="${pi/2} 0.0 0.0" /><!-- 116 = 90+52/2-->
+        <axis xyz="0.0 0.0 -1" />
+    </joint>
+    <link name="right_wheel_back_link">
+        <visual>
+            <geometry>
+                <cylinder radius="0.0625" length="0.05132" />
+            </geometry>
+            <material name="blue" />
+        </visual>
+        <collision>
+            <geometry>
+               <sphere radius="0.0625" />
+                <!-- <cylinder radius="0.0625" length="0.05132" /> -->
+            </geometry>
+            <!-- <material name="orange" /> -->
+        </collision>
+        <xacro:inertial_cylinder mass="0.1" length="0.04" radius="0.05">
+            <origin xyz="0 0 0" rpy="0 0 0" />
+        </xacro:inertial_cylinder>
+    </link>
+    <gazebo reference="right_wheel_back_link">
+        <material>Gazebo/Blue</material>
+    </gazebo>
+    <!--LEFT
+    WHEEL FOWARD LINK-->
+    <joint name="left_wheel_foward_joint" type="fixed">
+        <parent link="base_link" />
+        <child link="left_wheel_foward_link" />
+        <origin xyz="0.075 0.116 0.0" rpy="-${pi/2} 0.0 0.0" /><!-- 116 = 90+52/2-->
+        <axis xyz="0.0 0.0 1" />
+    </joint>
+    <link name="left_wheel_foward_link">
+        <visual>
+            <geometry>
+                <cylinder radius="0.0625" length="0.05132" />
+            </geometry>
+            <material name="blue" />
+        </visual>
+        <collision>
+            <geometry>
+                <sphere radius="0.0625" />
+                <!-- <cylinder radius="0.0625" length="0.05132" /> -->
+            </geometry>
+            <!-- <material name="orange" /> -->
+        </collision>
+        <xacro:inertial_cylinder mass="0.1" length="0.04" radius="0.05">
+            <origin xyz="0 0 0" rpy="0 0 0" />
+        </xacro:inertial_cylinder>
+    </link>
+    <gazebo reference="left_wheel_foward_link">
+        <material>Gazebo/Blue</material>
+        <!-- <mu1 value="0.001" />
+        <mu2 value="0.001" /> -->
+    </gazebo>
+    <!--RIGHT
+    WHEEL FOWARD LINK-->
+    <joint name="right_wheel_foward_joint" type="fixed">
+        <parent link="base_link" />
+        <child link="right_wheel_foward_link" />
+        <origin xyz="0.075 -0.116 0.0" rpy="${pi/2} 0.0 0.0" /><!-- 116 = 90+52/2-->
+        <axis xyz="0.0 0.0 -1" />
+    </joint>
+    <link name="right_wheel_foward_link">
+        <visual>
+            <geometry>
+                <cylinder radius="0.0625" length="0.05132" />
+            </geometry>
+            <material name="blue" />
+        </visual>
+        <collision>
+            <geometry>
+              <sphere radius="0.0625" />
+                <!-- <cylinder radius="0.0625" length="0.05132" /> -->
+            </geometry>
+            <!-- <material name="orange" /> -->
+        </collision>
+        <xacro:inertial_cylinder mass="0.1" length="0.04" radius="0.05">
+            <origin xyz="0 0 0" rpy="0 0 0" />
+        </xacro:inertial_cylinder>
+    </link>
+    <gazebo reference="right_wheel_foward_link">
+        <material>Gazebo/Blue</material>
+        <!-- <mu1 value="0.001" />
+        <mu2 value="0.001" /> -->
+    </gazebo>
+</robot>

File: install/bbb_robot/share/bbb_robot/description/ros2_control.xacro (robot description, xacro)
@@ -1 +1,61 @@
-/home/jetson/bbb_jetson_ws/src/bbb_robot/description/ros2_control.xacro
+<?xml version="1.0"?>
+<robot xmlns:xacro="http://www.ros.org/wiki/xacro">
+    <!-- <ros2_control name="GazeboSystem" type="system">
+        <hardware>
+            <plugin>gazebo_ros2_control/GazeboSystem</plugin>
+        </hardware>
+        <joint name="left_wheel_back_joint">
+            <command_interface name="velocity">
+                <param name="min">-10</param>
+                <param name="max"> 10</param>
+            </command_interface>
+            <state_interface name="velocity" />
+            <state_interface name="position" />
+        </joint>
+        <joint name="right_wheel_back_joint">
+            <command_interface name="velocity">
+                <param name="min">-10</param>
+                <param name="max"> 10</param>
+            </command_interface>
+            <state_interface name="velocity" />
+            <state_interface name="position" />
+        </joint>
+    </ros2_control> -->
+    <ros2_control name="Real_robot" type="system">
+        <hardware>
+            <plugin>diffdrive_arduino/DiffDriveArduino</plugin>
+            <param name="left_wheel_name">left_wheel_back_joint"</param>
+            <param name="right_wheel_name">right_wheel_back_joint</param>
+            <param name="loop_rate">30</param>
+            <param name="device">/dev/ttyUSB0</param>
+            <param name="baud_rate">57600</param>
+            <param name="timeout">1000</param>
+            <param name="enc_counts_per_rev">3436</param>
+        </hardware>
+        <joint name="left_wheel_back_joint">
+            <command_interface name="velocity">
+                <param name="min">-10</param>
+                <param name="max"> 10</param>
+            </command_interface>
+            <state_interface name="velocity" />
+            <state_interface name="position" />
+        </joint>
+        <joint name="right_wheel_back_joint">
+            <command_interface name="velocity">
+                <param name="min">-10</param>
+                <param name="max"> 10</param>
+            </command_interface>
+            <state_interface name="velocity" />
+            <state_interface name="position" />
+        </joint>
+    </ros2_control>
+    <!-- <gazebo>
+        <plugin name="gazebo_ros2_control" filename="libgazebo_ros2_control.so">
+            <parameters>$(find bbb_robot)/config/my_controllers.yaml</parameters>
+        </plugin>
+    </gazebo> -->
+</robot>
+<!-- ros2 run teleop_twist_keyboard teleop_twist_keyboard -->
+<!-- teleop: stands for teleoperation
+twist: type of date, ros uused to express linear velocity and angle
+keyboard: use keyboard to control remote robot -->
